File: SplitFlapBusBoard/SplitFlapBusBoard.kicad_pcb (KiCad board)
At the start: 2 copper layers, 456 x 12 mm, 2 parts, among them J1 Conn_01x04_Pin, J2 Conn_01x04_Pin

Commit message: Version 2 of Hub and Module Board
Finished and ordered bus board and V2 or Module board (50x)
Parts:
- removed J1: Conn_01x04_Pin, Connector_PinHeader_2.54mm:PinHeader_1x04_P2.54mm_Vertical
- moved J2 78.8 mm to (20.0, 20.0)
Connections:
- J2 pad 1: +5V -> +12V
- J2 pad 2: GND -> A
- J2 pad 3: /B -> B
- J2 pad 4: /A -> GND
Routing:
- net /A: track 7.54 -> 0.00 mm
- net GND: track 7.53 -> 0.00 mm, vias 20 -> 0
- net /B: track 7.53 -> 0.00 mm
- net +5V: track 7.53 -> 0.00 mm
Other:
- board size 456 x 12 mm -> 572.6 x 24 mm
- board text added: "12V A B GND"
